File: hardware/swc_wing/swc_wing.kicad_sch (KiCad schematic)
At the start: 53 parts, among them J1 Conn_01x06_Female, J3 Conn_01x06_Female, J4 Conn_01x01_Female, Q1 2N7002, Q2 2N7002, Q3 2N7002, Q4 2N7002, Q5 2N7002, SW1 SW_Push_LED, SW2 SW_Push_LED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

Commit message: 3.3v-ify wing
Parts:
- J2: renamed from J?; footprint Connector_PinHeader_2.54mm:PinHeader_1x06_P2.54mm_Horizontal -> Connector_PinHeader_2.54mm:PinHeader_1x05_P2.54mm_Horizontal
- gave numbers to parts that had none: 2
Connections:
- net +3.3V: now also J4.1 (Pin_1), R6.2, R7.2, R8.2, U2.3 (A0), U3.4 (A1)
- net +5V: no longer J4.1 (Pin_1), R6.2, R7.2, R8.2, U2.3 (A0), U3.4 (A1)
