File: hardware/swc/swc.kicad_pcb (KiCad board)
At the start: 4 copper layers, 53.5 x 53.5 mm, 60 parts, among them J1 Conn_01x04_Female, J2 Conn_02x10_Odd_Even, J3 Conn_01x05, J4 FTSH-107-01-F-DV-K, J5 Conn_01x05, J6 Conn_01x03, U1 TJA1051T-3, U2 LMR14020, U3 XC6206P332MR, U4 STM32F042C6Tx

Commit message: missing lcsc
Changed lines of the file:
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@@
     (fp_line (start -2.45 -2.35) (end -2.45 3.4) (layer "F.Fab") (width 0.1))
     (fp_line (start 12.45 3.4) (end 12.45 -2.35) (layer "F.Fab") (width 0.1))
-    (pad "1" thru_hole roundrect (at 0 0 90) (size 1.7 1.95) (drill 0.95) (layers *.Cu *.Mask) (roundrect_rratio 0.147059)
+    (pad "1" thru_hole roundrect (at 0 0 90) (size 1.7 1.95) (drill 0.95) (layers *.Cu *.Mask) (roundrect_rratio 0.1470588235)
       (net 3 "+5V") (pinfunction "Pin_1") (pintype "passive"))
     (pad "2" thru_hole oval (at 2.5 0 90) (size 1.7 1.95) (drill 0.95) (layers *.Cu *.Mask)
@@
     (fp_line (start -1 0.625) (end -1 -0.625) (layer "F.Fab") (width 0.1))
     (fp_line (start 1 -0.625) (end 1 0.625) (layer "F.Fab") (width 0.1))
-    (pad "1" smd roundrect (at -0.9125 0) (size 1.025 1.4) (layers "F.Cu" "F.Paste" "F.Mask") (roundrect_rratio 0.243902)
+    (pad "1" smd roundrect (at -0.9125 0) (size 1.025 1.4) (layers "F.Cu" "F.Paste" "F.Mask") (roundrect_rratio 0.243902439)
       (net 68 "CANH") (pintype "passive"))
-    (pad "2" smd roundrect (at 0.9125 0) (size 1.025 1.4) (layers "F.Cu" "F.Paste" "F.Mask") (roundrect_rratio 0.243902)
+    (pad "2" smd roundrect (at 0.9125 0) (size 1.025 1.4) (layers "F.Cu" "F.Paste" "F.Mask") (roundrect_rratio 0.243902439)
       (net 69 "CANL") (pintype "passive"))
     (model "${KICAD6_3DMODEL_DIR}/Resistor_SMD.3dshapes/R_0805_2012Metric.wrl"
@@
     (fp_line (start -2.45 -2.35) (end -2.45 3.4) (layer "F.Fab") (width 0.1))
     (fp_line (start -0.625 -2.35) (end 0 -1.35) (layer "F.Fab") (width 0.1))
-    (pad "1" thru_hole roundrect (at 0 0 270) (size 1.7 1.95) (drill 0.95) (layers *.Cu *.Mask) (roundrect_rratio 0.147059)
+    (pad "1" thru_hole roundrect (at 0 0 270) (size 1.7 1.95) (drill 0.95) (layers *.Cu *.Mask) (roundrect_rratio 0.1470588235)
       (net 3 "+5V") (pinfunction "Pin_1") (pintype "passive"))
     (pad "2" thru_hole oval (at 2.5 0 270) (size 1.7 1.95) (drill 0.95) (layers *.Cu *.Mask)
@@
     (fp_line (start 0 1.35) (end 0.625 2.35) (layer "B.Fab") (width 0.1))
     (fp_line (start 9.95 2.35) (end -2.45 2.35) (layer "B.Fab") (width 0.1))
-    (pad "1" thru_hole roundrect (at 0 0) (size 1.7 1.95) (drill 0.95) (layers *.Cu *.Mask) (roundrect_rratio 0.147059)
+    (pad "1" thru_hole roundrect (at 0 0) (size 1.7 1.95) (drill 0.95) (layers *.Cu *.Mask) (roundrect_rratio 0.1470588235)
       (net 6 "+12V") (pinfunction "Pin_1") (pintype "passive"))
     (pad "2" thru_hole oval (at 2.5 0) (size 1.7 1.95) (drill 0.95) (layers *.Cu *.Mask)

Commit message: close to final main board
Parts:
- removed RN3: 470k, Resistor_SMD:R_Array_Convex_4x0603
- added J7: Conn_ARM_SWD_TagConnect_TC2030-NL, Connector:Tag-Connect_TC2030-IDC-NL_2x03_P1.27mm_Vertical, F.Cu at (50.2, 41.5)
- added R5: 470k, Resistor_SMD:R_0402_1005Metric, F.Cu at (44.7, 60.0)
- added R6: 470k, Resistor_SMD:R_0402_1005Metric, F.Cu at (44.7, 58.9)
- added R7: 470k, Resistor_SMD:R_0402_1005Metric, F.Cu at (44.7, 57.8)
- added R8: 470k, Resistor_SMD:R_0402_1005Metric, F.Cu at (44.7, 56.7)
- D7: footprint Package_TO_SOT_SMD:SOT-23 -> Package_TO_SOT_SMD:SOT-323_SC-70
- moved D7 0.11 mm to (40.8, 32.4)
Routing:
- net SWCLK: track 14.7 -> 63.6 mm, vias 2 -> 4
- net SWDIO: track 14.5 -> 62.6 mm, vias 2 -> 4
- net nRESET: track 18.0 -> 54.3 mm, vias 2 -> 3
- net +3V3: track 136.2 -> 141.0 mm
- net Net-(J2-Pad10): track 20.7 -> 21.5 mm
- net Net-(J2-Pad16): track 18.6 -> 18.1 mm
- net GND: vias 142 -> 144
Other:
- board text added: "github.com/mck1117/swc"
- board text added: "rev.a 20230807"

Commit message: drc
Parts:
- moved TP1 0.25 mm to (30.9, 32.5)
Connections:
- U1 pad 8: unconnected-(U1-Pad8) -> GND
Changed lines of the file:
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@@
   (net 65 "Net-(R16-Pad2)")
   (net 66 "Net-(TP1-Pad1)")
-  (net 67 "unconnected-(U1-Pad8)")
-  (net 68 "CANH")
-  (net 69 "CANL")
-  (net 70 "unconnected-(J7-Pad6)")
+  (net 67 "CANH")
+  (net 68 "CANL")
+  (net 69 "unconnected-(J7-Pad6)")
   (footprint "Diode_SMD:D_SMA" (layer "F.Cu")
     (at 32.3 23.1)
@@
     (fp_line (start 1 -0.625) (end 1 0.625) (layer "F.Fab") (width 0.1))
     (pad "1" smd roundrect (at -0.9125 0) (size 1.025 1.4) (layers "F.Cu" "F.Paste" "F.Mask") (roundrect_rratio 0.243902439)
-      (net 68 "CANH") (pintype "passive"))
+      (net 67 "CANH") (pintype "passive"))
     (pad "2" smd roundrect (at 0.9125 0) (size 1.025 1.4) (layers "F.Cu" "F.Paste" "F.Mask") (roundrect_rratio 0.243902439)
-      (net 69 "CANL") (pintype "passive"))
+      (net 68 "CANL") (pintype "passive"))
     (model "${KICAD6_3DMODEL_DIR}/Resistor_SMD.3dshapes/R_0805_2012Metric.wrl"
       (offset (xyz 0 0 0))
@@
       (net 2 "GND") (pinfunction "GND") (pintype "power_in"))
     (pad "6" connect circle (at 1.27 -0.635 270) (size 0.7874 0.7874) (layers "F.Cu" "F.Mask")
-      (net 70 "unconnected-(J7-Pad6)") (pinfunction "SWO") (pintype "input+no_connect"))
+      (net 69 "unconnected-(J7-Pad6)") (pinfunction "SWO") (pintype "input+no_connect"))
     (zone (net 0) (net_name "") (layer "F.Cu") (hatch full 0.508)
       (connect_pads (clearance 0))
@@
     (fp_line (start -0.68 -0.6) (end -0.68 1.1) (layer "F.Fab") (width 0.1))
     (pad "1" smd rect (at -1 -0.65 180) (size 0.45 0.7) (layers "F.Cu" "F.Paste" "F.Mask")
-      (net 69 "CANL") (pinfunction "A1") (pintype "passive"))
+      (net 68 "CANL") (pinfunction "A1") (pintype "passive"))
     (pad "2" smd rect (at -1 0.65 180) (size 0.45 0.7) (layers "F.Cu" "F.Paste" "F.Mask")
-      (net 68 "CANH") (pinfunction "A2") (pintype "passive"))
+      (net 67 "CANH") (pinfunction "A2") (pintype "passive"))
     (pad "3" smd rect (at 1 0 180) (size 0.45 0.7) (layers "F.Cu" "F.Paste" "F.Mask")
       (net 2 "GND") (pinfunction "common") (pintype "input"))
@@
       (net 4 "+3V3") (pinfunction "VIO") (pintype "power_in"))
     (pad "6" smd roundrect (at 2.475 0.635 180) (size 1.95 0.6) (layers "F.Cu" "F.Paste" "F.Mask") (roundrect_rratio 0.25)
-      (net 69 "CANL") (pinfunction "CANL") (pintype "bidirectional"))
+      (net 68 "CANL") (pinfunction "CANL") (pintype "bidirectional"))
     (pad "7" smd roundrect (at 2.475 -0.635 180) (size 1.95 0.6) (layers "F.Cu" "F.Paste" "F.Mask") (roundrect_rratio 0.25)
-      (net 68 "CANH") (pinfunction "CANH") (pintype "bidirectional"))
+      (net 67 "CANH") (pinfunction "CANH") (pintype "bidirectional"))
     (pad "8" smd roundrect (at 2.475 -1.905 180) (size 1.95 0.6) (layers "F.Cu" "F.Paste" "F.Mask") (roundrect_rratio 0.25)
-      (net 67 "unconnected-(U1-Pad8)") (pinfunction "S") (pintype "input"))
+      (net 2 "GND") (pinfunction "S") (pintype "input"))
     (model "${KICAD6_3DMODEL_DIR}/Package_SO.3dshapes/SOIC-8_3.9x4.9mm_P1.27mm.wrl"
       (offset (xyz 0 0 0))
@@
   )
   (footprint "TestPoint:TestPoint_Pad_1.5x1.5mm" (layer "B.Cu")
-    (at 31.05 32.4 180)
+    (at 30.85 32.55 180)
     (descr "SMD rectangular pad as test Point, square 1.5mm side length")
     (tags "test point SMD pad rectangle square")
@@
       (net 6 "+12V") (pinfunction "Pin_1") (pintype "passive"))
     (pad "2" thru_hole oval (at 2.5 0) (size 1.7 1.95) (drill 0.95) (layers *.Cu *.Mask)
-      (net 68 "CANH") (pinfunction "Pin_2") (pintype "passive"))
+      (net 67 "CANH") (pinfunction "Pin_2") (pintype "passive"))
     (pad "3" thru_hole oval (at 5 0) (size 1.7 1.95) (drill 0.95) (layers *.Cu *.Mask)
-      (net 69 "CANL") (pinfunction "Pin_3") (pintype "passive"))
+      (net 68 "CANL") (pinfunction "Pin_3") (pintype "passive"))
     (pad "4" thru_hole oval (at 7.5 0) (size 1.7 1.95) (drill 0.95) (layers *.Cu *.Mask)
       (net 2 "GND") (pinfunction "Pin_4") (pintype "passive"))
@@
   (gr_circle (center 38.5 36.5) (end 65.25 36.5) (layer "Edge.Cuts") (width 0.25) (fill none))
   (gr_circle (center 38.5 36.5) (end 38.5 23.5) (layer "B.CrtYd") (width 0.05) (fill none))
-  (gr_text "LEDCLK" (at 34.3 32.25) (layer "B.SilkS")
+  (gr_text "LEDCLK" (at 34.25 32.5) (layer "B.SilkS")
     (effects (font (size 1 0.8) (thickness 0.12)) (justify mirror))
   )
@@
   (segment (start 28.2 23.01) (end 28.2 24.075) (width 0.25) (layer "F.Cu") (net 1))
   (via (at 23.3 27.3) (size 0.5) (drill 0.3) (layers "F.Cu" "B.Cu") (net 2))
-  (via (at 32.8 33.2) (size 0.5) (drill 0.3) (layers "F.Cu" "B.Cu") (net 2))
+  (via (at 32.9 33.3) (size 0.5) (drill 0.3) (layers "F.Cu" "B.Cu") (net 2))
   (via (at 22.75 37.65) (size 0.5) (drill 0.3) (layers "F.Cu" "B.Cu") (net 2))
   (via (at 40.8 26.9) (size 0.5) (drill 0.3) (layers "F.Cu" "B.Cu") (net 2))
@@
   (via (at 50 13.8) (size 0.5) (drill 0.3) (layers "F.Cu" "B.Cu") (net 2))
   (via (at 22.8 39) (size 0.5) (drill 0.3) (layers "F.Cu" "B.Cu") (net 2))
-  (via (at 32.2 33.2) (size 0.5) (drill 0.3) (layers "F.Cu" "B.Cu") (net 2))
+  (via (at 32.3 33.25) (size 0.5) (drill 0.3) (layers "F.Cu" "B.Cu") (net 2))
   (via (at 49.432376 16.177971) (size 0.5) (drill 0.3) (layers "F.Cu" "B.Cu") (net 2))
   (via (at 24.75 40.2) (size 0.5) (drill 0.3) (layers "F.Cu" "B.Cu") (net 2))
@@
   (segment (start 24.25 41.325) (end 24.225 41.3) (width 0.25) (layer "F.Cu") (net 4))
   (segment (start 13.3 39.9) (end 13.3 38.575) (width 0.2) (layer "F.Cu") (net 4))
-  (segment (start 45.7 52.3) (end 45.5 52.5) (width 0.75) (layer "F.Cu") (net 4))
   (segment (start 13.3 38.575) (end 14.2 37.675) (width 0.2) (layer "F.Cu") (net 4))
   (via (at 46.25 34.9) (size 0.75) (drill 0.45) (layers "F.Cu" "B.Cu") (net 4))
@@
   (segment (start 29.2 31.4) (end 30.35 31.4) (width 0.2) (layer "F.Cu") (net 66))
   (via (at 30.65 33.9) (size 0.5) (drill 0.3) (layers "F.Cu" "B.Cu") (net 66))
-  (segment (start 31.05 32.4) (end 31.05 33.5) (width 0.25) (layer "B.Cu") (net 66))
-  (segment (start 31.05 33.5) (end 30.65 33.9) (width 0.25) (layer "B.Cu") (net 66))
-  (segment (start 45.2 34.8) (end 45.2 36) (width 0.25) (layer "F.Cu") (net 68))
-  (segment (start 41.0375 36.35) (end 39.8875 35.2) (width 0.25) (layer "F.Cu") (net 68))
-  (segment (start 40.15 32.2) (end 39.8875 32.4625) (width 0.25) (layer "F.Cu") (net 68))
-  (segment (start 40.15 31.4) (end 40.15 32.2) (width 0.25) (layer "F.Cu") (net 68))
-  (segment (start 45.2 36) (end 44.85 36.35) (width 0.25) (layer "F.Cu") (net 68))
-  (segment (start 40 31.4) (end 40.15 31.4) (width 0.25) (layer "F.Cu") (net 68))
-  (segment (start 44.85 36.35) (end 41.0375 36.35) (width 0.25) (layer "F.Cu") (net 68))
-  (segment (start 44.635 34.235) (end 45.2 34.8) (width 0.25) (layer "F.Cu") (net 68))
-  (segment (start 37.6 29) (end 40 31.4) (width 0.25) (layer "F.Cu") (net 68))
-  (segment (start 39.8875 32.4625) (end 39.8875 35.2) (width 0.25) (layer "F.Cu") (net 68))
-  (segment (start 43.825 34.235) (end 44.635 34.235) (width 0.25) (layer "F.Cu") (net 68))
-  (segment (start 41.7 35.1875) (end 41.7125 35.2) (width 0.25) (layer "F.Cu") (net 69))
-  (segment (start 41.715 32.965) (end 41.7 32.95) (width 0.25) (layer "F.Cu") (net 69))
-  (segment (start 40.1 29) (end 41.45 30.35) (width 0.25) (layer "F.Cu") (net 69))
-  (segment (start 41.7 32.95) (end 41.7 35.1875) (width 0.25) (layer "F.Cu") (net 69))
-  (segment (start 41.45 32.7) (end 41.45 31.4) (width 0.25) (layer "F.Cu") (net 69))
-  (segment (start 41.7 32.95) (end 41.45 32.7) (width 0.25) (layer "F.Cu") (net 69))
-  (segment (start 43.825 32.965) (end 41.715 32.965) (width 0.25) (layer "F.Cu") (net 69))
-  (segment (start 41.45 30.35) (end 41.45 31.4) (width 0.25) (layer "F.Cu") (net 69))
+  (segment (start 30.65 32.75) (end 30.85 32.55) (width 0.25) (layer "B.Cu") (net 66))
+  (segment (start 30.65 33.9) (end 30.65 32.75) (width 0.25) (layer "B.Cu") (net 66))
+  (segment (start 45.2 34.8) (end 45.2 36) (width 0.25) (layer "F.Cu") (net 67))
+  (segment (start 41.0375 36.35) (end 39.8875 35.2) (width 0.25) (layer "F.Cu") (net 67))
+  (segment (start 40.15 32.2) (end 39.8875 32.4625) (width 0.25) (layer "F.Cu") (net 67))
+  (segment (start 40.15 31.4) (end 40.15 32.2) (width 0.25) (layer "F.Cu") (net 67))
+  (segment (start 45.2 36) (end 44.85 36.35) (width 0.25) (layer "F.Cu") (net 67))
+  (segment (start 40 31.4) (end 40.15 31.4) (width 0.25) (layer "F.Cu") (net 67))
+  (segment (start 44.85 36.35) (end 41.0375 36.35) (width 0.25) (layer "F.Cu") (net 67))
+  (segment (start 44.635 34.235) (end 45.2 34.8) (width 0.25) (layer "F.Cu") (net 67))
+  (segment (start 37.6 29) (end 40 31.4) (width 0.25) (layer "F.Cu") (net 67))
+  (segment (start 39.8875 32.4625) (end 39.8875 35.2) (width 0.25) (layer "F.Cu") (net 67))
+  (segment (start 43.825 34.235) (end 44.635 34.235) (width 0.25) (layer "F.Cu") (net 67))
+  (segment (start 41.7 35.1875) (end 41.7125 35.2) (width 0.25) (layer "F.Cu") (net 68))
+  (segment (start 41.715 32.965) (end 41.7 32.95) (width 0.25) (layer "F.Cu") (net 68))
+  (segment (start 40.1 29) (end 41.45 30.35) (width 0.25) (layer "F.Cu") (net 68))
+  (segment (start 41.7 32.95) (end 41.7 35.1875) (width 0.25) (layer "F.Cu") (net 68))
+  (segment (start 41.45 32.7) (end 41.45 31.4) (width 0.25) (layer "F.Cu") (net 68))
+  (segment (start 41.7 32.95) (end 41.45 32.7) (width 0.25) (layer "F.Cu") (net 68))
+  (segment (start 43.825 32.965) (end 41.715 32.965) (width 0.25) (layer "F.Cu") (net 68))
+  (segment (start 41.45 30.35) (end 41.45 31.4) (width 0.25) (layer "F.Cu") (net 68))
   (zone (net 62) (net_name "Net-(C13-Pad2)") (layer "F.Cu") (hatch edge 0.508)
     (priority 1)

Commit message: main board export
Parts:
- L2: value 10u -> 8.2u; footprint mwsa0503:MWSA0503 -> Inductor_SMD:L_Bourns_SRN6045TA
- moved C22 10.3 mm to (54.4, 23.6), turned to 0 degrees
- moved C21 2.15 mm to (47.2, 16.4), turned to 180 degrees
- moved L2 1.14 mm to (48.5, 20.9), turned to 0 degrees
- moved C13 0.89 mm to (37.0, 20.4)
- moved D6 0.85 mm to (41.4, 20.4)
Routing:
- net +5V: track 11.8 -> 1.63 mm, vias 10 -> 16
- net Net-(C13-Pad1): track 1.84 -> 3.22 mm
- net Net-(C2-Pad1): track 20.4 -> 19.8 mm
- net GND: vias 144 -> 166
