File: hardware/swc/swc.kicad_sch (KiCad schematic)
At the start: 60 parts, among them J1 Conn_01x04_Female, J2 Conn_02x10_Odd_Even, J3 Conn_01x05, J4 FTSH-107-01-F-DV-K, J5 Conn_01x05, J6 Conn_01x03, U1 TJA1051T-3, U2 LMR14020, U3 XC6206P332MR, U4 STM32F042C6Tx

Commit message: missing lcsc
Parts:
- D7: LCSC (none) -> C152727
Changed lines of the file:
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@@
+      (effects (font (size 1.27 1.27)) hide)
+    )
+    (property "LCSC" "C152727" (id 4) (at 161.925 180.975 0)
       (effects (font (size 1.27 1.27)) hide)
     )

Commit message: close to final main board
Parts:
- removed RN3: 470k, Resistor_SMD:R_Array_Convex_4x0603, symbol Device:R_Pack04
- added J7: Conn_ARM_SWD_TagConnect_TC2030-NL, Connector:Tag-Connect_TC2030-IDC-NL_2x03_P1.27mm_Vertical, symbol Connector:Conn_ARM_SWD_TagConnect_TC2030-NL
- added R5, R6, R7, R8: 470k, Resistor_SMD:R_0402_1005Metric, symbol Device:R
- D7: footprint Package_TO_SOT_SMD:SOT-23 -> Package_TO_SOT_SMD:SOT-323_SC-70
Connections:
- net +3V3: now also J7.1 (VCC)
- net GND: now also J7.5 (GND), R5.2, R6.2, R7.2, R8.2
- net SWCLK: now also J7.4 (SWCLK)
- net SWDIO: now also J7.2 (SWDIO)
- net nRESET: now also J7.3 (~{RESET})
- net at J2.10 (Pin_10), RN5.5 (R4.2): now also R5.1
- net at J2.12 (Pin_12), RN5.6 (R3.2): now also R6.1
- net at J2.14 (Pin_14), RN5.7 (R2.2): now also R7.1
- net at J2.16 (Pin_16), RN5.8 (R1.2): now also R8.1
- no-connect marks 19 -> 20

Commit message: erc
Connections:
- net GND: now also U1.8 (S)
Changed lines of the file:
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@@
     (pin "2")
+  )
+  (symbol (lib_id "power:GND") (at 118.11 186.055 270) (unit 1)
+    (in_bom yes) (on_board yes) (fields_autoplaced)
+    (property "Reference" "#PWR0163" (id 0) (at 111.76 186.055 0)
+      (effects (font (size 1.27 1.27)) hide)
+    )
+    (property "Value" "GND" (id 1) (at 113.665 186.055 0)
+      (effects (font (size 1.27 1.27)) hide)
+    )
+    (property "Footprint" "" (id 2) (at 118.11 186.055 0)
+      (effects (font (size 1.27 1.27)) hide)
+    )
+    (property "Datasheet" "" (id 3) (at 118.11 186.055 0)
+      (effects (font (size 1.27 1.27)) hide)
+    )
+    (pin "1")
   )
   (symbol (lib_id "power:+3.3V") (at 220.345 129.54 0) (unit 1)
@@
       (reference "#PWR0162") (unit 1) (value "GND") (footprint "")
     )
+    (path "/198bd8cd-6415-48ae-8a41-c221492053fb"
+      (reference "#PWR0163") (unit 1) (value "GND") (footprint "")
+    )
     (path "/27657bad-e009-4803-bfa1-449a6cddb759"

Commit message: main board export
Parts:
- L2: value 10u -> 8.2u; footprint mwsa0503:MWSA0503 -> Inductor_SMD:L_Bourns_SRN6045TA; LCSC C408412 -> (none); LCSC_ext 1 -> (none); possible_not_ext 1 -> (none)
Changed lines of the file:
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@@
     (in_bom yes) (on_board yes)
     (property "Reference" "L2" (id 0) (at 146.05 33.02 90))
-    (property "Value" "10u" (id 1) (at 146.685 30.734 90))
-    (property "Footprint" "mwsa0503:MWSA0503" (id 2) (at 146.685 35.56 0)
+    (property "Value" "8.2u" (id 1) (at 146.685 30.734 90))
+    (property "Footprint" "Inductor_SMD:L_Bourns_SRN6045TA" (id 2) (at 146.685 35.56 0)
       (effects (font (size 1.27 1.27)) hide)
     )
@@
       (effects (font (size 1.27 1.27)) hide)
     )
-    (property "LCSC" "C408412" (id 5) (at 146.685 35.56 0)
-      (effects (font (size 1.27 1.27)) hide)
-    )
-    (property "LCSC_ext" "1" (id 6) (at 146.685 35.56 0)
-      (effects (font (size 1.27 1.27)) hide)
-    )
-    (property "possible_not_ext" "1" (id 7) (at 146.685 35.56 0)
+    (property "LCSC" "" (id 5) (at 146.685 35.56 0)
+      (effects (font (size 1.27 1.27)) hide)
+    )
+    (property "LCSC_ext" "" (id 6) (at 146.685 35.56 0)
+      (effects (font (size 1.27 1.27)) hide)
+    )
+    (property "possible_not_ext" "" (id 7) (at 146.685 35.56 0)
       (effects (font (size 1.27 1.27)) hide)
     )
@@
     )
     (path "/c6cb152f-1598-48c6-b75e-07c363e4d342"
-      (reference "L2") (unit 1) (value "10u") (footprint "mwsa0503:MWSA0503")
+      (reference "L2") (unit 1) (value "8.2u") (footprint "Inductor_SMD:L_Bourns_SRN6045TA")
     )
     (path "/273d054b-2420-4688-835b-4223b20c0a8c"
